Commit message: [1.0.1] Final URDF done

File: urdf/rosbot3.xacro (robot description, xacro)
@@ -5,8 +5,9 @@
 -->
 <robot name="rosbot3" xmlns:xacro="http://www.ros.org/wiki/xacro">
-  <xacro:include filename="$(find rosbot3_description)/urdf/ugv02.xacro"/>
+  <xacro:include filename="$(find rosbot3_description)/urdf/rosbot3_body.xacro"/>
   <xacro:property name="overall_height_with_lidar" value="${141.0 * M}"/>
   <xacro:property name="overall_height_with_camera" value="${197.0 * M}"/>
   <!--
+    Rosbot3 Lidar Properties
     RosBot3 Lidar (Rosbot3 Pro Lidar is different)
     https://www.slamtec.com/en/C1/Spec
@@ -18,4 +19,5 @@
   <xacro:property name="lidar_radius" value="${lidar_side * 0.4}"/>
   <!--
+    Rosbot3 Camera Properties
     Rosbot3 Camera (Rosbot3 Pro Camera is different)
     https://shop.luxonis.com/products/oak-d-lite-1?variant=42583102456031
@@ -27,77 +29,16 @@
   <xacro:property name="camera_square_base_thickness" value="${1.0 * M}"/>
   <!--
-    Value calculated considering heigths with and without camera and a 45° angle starting from the base
-    Calculus -> (overall_height_with_camera-overall_height-camera_height*0.5 - camera_square_base_thickness)/ (sine(45°))
+    Value calculated considering heigths with and without camera and a 30° angle starting from the base
+    Calculus -> (overall_height_with_camera-overall_height-camera_height*0.5 - camera_square_base_thickness)/ (cos(30°))
   -->
-  <xacro:property name="camera_square_stem_length" value="${(overall_height_with_camera - overall_height - camera_heigth * 0.2 - camera_square_base_thickness ) * (sqrt(2)/2.0) }"/>
+  <xacro:property name="camera_square_stem_length" value="${(overall_height_with_camera - overall_height - camera_heigth * 0.5 - camera_square_base_thickness ) * (2/sqrt(3)) }"/>
   <!--
-    Rosbot3 Camera (Rosbot3 Pro Camera is different)
-    https://shop.luxonis.com/products/oak-d-lite-1?variant=42583102456031
-    Need to fix camera front, its no accurate
+    Wifi Antenna Properties
   -->
-  <xacro:macro
-    name="camera_base"
-  >
-    <xacro:solid_block
-      name="camera_left_square_base"
-      size_x="${camera_square_base_side}"
-      size_y="${camera_square_base_side}"
-      size_z="${camera_square_base_thickness}"
-      yaw="${45 * DEG}"
-    />
-    <xacro:solid_block
-      name="camera_left_stem"
-      size_x="${camera_square_base_side * 0.5}"
-      size_y="${camera_square_base_side * 0.5}"
-      size_z="${camera_square_stem_length}"
-      pitch="${45 * DEG}"
-    />
-    <xacro:joint_fixed
-      parent="camera_left_square_base"
-      child="camera_left_stem"
-      z="${(camera_square_base_thickness + camera_square_stem_length * sqrt(2) * 0.5) * 0.5}"
-      x="${(camera_square_stem_length * sqrt(2) * 0.5) * 0.5}"
-    />
-    <!-- <xacro:solid_cylinder
-      name="wheel_${position}_right"
-      length="${wheel_thickness}"
-      radius="${wheel_radius}"
-      roll="${90.0 * DEG}"
-    />
-    <xacro:solid_cylinder
-      name="wheel_${position}_axle"
-      length="${body_width}"
-      radius="0.005"
-      roll="${90.0 * DEG}"
-    />
-    <xacro:joint_continuous
-      name="joint_wheel_${position}_left"
-      parent="wheel_${position}_axle"
-      child="wheel_${position}_left"
-      y="${(body_width + wheel_thickness) * 0.5}"
-      axis="0 1 0"
-    />
-    <xacro:joint_continuous
-      name="joint_wheel_${position}_right"
-      parent="wheel_${position}_axle"
-      child="wheel_${position}_right"
-      y="${(body_width + wheel_thickness) * -0.5}"
-      axis="0 1 0"
-    /> -->
-  </xacro:macro>
-  <!-- <xacro:camera_base/>
-  <xacro:joint_fixed
-    parent="fenders_top"
-    child="camera_left_square_base"
-    x="${-lidar_side*0.5 - camera_square_stem_length* (1/math.sqrt(2)) }"
-    y="${-lidar_side * 0.5}"
-    z="${(fender_thickness + camera_square_base_thickness) * 0.5}"
-  /> -->
-  <link name="camera_front"/>
-  <xacro:joint_fixed
-    parent="fenders_top"
-    child="camera_front"
-    x="${0.5 * fender_thickness}"
-  />
+  <!-- Scaling Wifi Antenna by 1.2-->
+  <xacro:property name="wifi_antenna_length" value="${ ((overall_height_with_camera - overall_height)*0.5) *1.2}"/>
+  <xacro:property name="wifi_antenna_radius" value="${3 * M}"/>
+  <xacro:property name="wifi_antenna_distance_x_offset_from_camera" value="${80 * M}"/>
+  <xacro:property name="wifi_antenna_distance_z_offset_from_camera" value="${overall_height_with_camera - overall_height - camera_heigth *0.5 }"/>
   <!--
     RosBot3 Lidar (Rosbot3 Pro Lidar is different)
@@ -135,3 +76,96 @@
     z="${lidar_base_height + lidar_height * 0.5}"
   />
+  <!--
+    Rosbot3 Camera (Rosbot3 Pro Camera is different)
+    https://shop.luxonis.com/products/oak-d-lite-1?variant=42583102456031
+    Camera Base is arbitrary, made equal as much as possible to the model, without making too much complex TFs
+  -->
+  <!--
+    Camera base macro, since it has two different fixation rods
+  -->
+  <xacro:macro
+    name="camera_base"
+    params="position"
+  >
+ <xacro:solid_block
+    name="camera_up_${position}_stem"
+    size_x="${camera_square_base_side * 0.5}"
+    size_y="${camera_square_base_side * 0.5}"
+    size_z="${0.5 * lidar_side - camera_thickness }"
+    pitch="${90.0 * DEG}"
+  />
+  <xacro:solid_block
+    name="camera_down_${position}_stem"
+    size_x="${camera_square_base_side * 0.5}"
+    size_y="${camera_square_base_side * 0.5}"
+    size_z="${camera_square_stem_length}"
+    pitch="${30.0 * DEG}"
+  />
+  <xacro:solid_block
+    name="camera_${position}_square_base"
+    size_x="${camera_square_base_side}"
+    size_y="${camera_square_base_side}"
+    size_z="${camera_square_base_thickness}"
+    yaw="${45 * DEG}"
+  />
+  <xacro:joint_fixed
+    parent="camera_up_${position}_stem"
+    child="camera_down_${position}_stem"
+    x="${-0.5 * (camera_square_base_side* 0.5 + 0.5 * lidar_side - camera_thickness + camera_square_stem_length * 0.5) + camera_square_base_side* 0.5}"
+    z="${-0.5 * (camera_square_stem_length * (sqrt(3)/2)- camera_square_base_side * 0.5)}"
+  />
+  <xacro:joint_fixed
+    parent="camera_down_${position}_stem"
+    child="camera_${position}_square_base"
+    x="${-0.5 * (camera_square_stem_length*0.5)}"
+    z="${-0.5 * (camera_square_stem_length *(sqrt(3)/2) + camera_square_base_thickness)}"
+  />
+  </xacro:macro>
+  <xacro:solid_block
+    name="camera"
+    size_x="${camera_thickness}"
+    size_y="${camera_length}"
+    size_z="${camera_heigth}"
+  />
+  <xacro:joint_fixed
+    parent="lidar"
+    child="camera"
+    z="${0.5 * (lidar_height-camera_heigth) + overall_height_with_camera - overall_height_with_lidar}"
+    x="${-0.5 * camera_thickness}"
+  />
+  <link name="camera_front"/>
+  <xacro:joint_fixed
+    parent="camera"
+    child="camera_front"
+    x="${0.5 * camera_thickness}"
+  />
+  <xacro:camera_base position="left"/>
+  <xacro:camera_base position="right"/>
+  <xacro:joint_fixed
+    parent="camera"
+    child="camera_up_left_stem"
+    x="${-0.5 * (camera_thickness + 0.5 * lidar_side - camera_thickness)}"
+    y="${0.5 * (0.5 * camera_length)}"
+  />
+  <xacro:joint_fixed
+    parent="camera"
+    child="camera_up_right_stem"
+    x="${-0.5 * (camera_thickness + 0.5 * lidar_side - camera_thickness)}"
+    y="${-0.5 * (0.5 * camera_length)}"
+  />
+  <!--
+    Wifi Antenna
+  -->
+  <xacro:solid_cylinder
+    name="wifi_antenna"
+    length="${wifi_antenna_length}"
+    radius="${wifi_antenna_radius}"
+  />
+  <xacro:joint_fixed
+    parent="camera"
+    child="wifi_antenna"
+    x="${-(0.5 * camera_thickness + wifi_antenna_distance_x_offset_from_camera - wifi_antenna_radius) }"
+    y="${0.5 * camera_length}"
+    z="${0.5 * wifi_antenna_length - wifi_antenna_distance_z_offset_from_camera}"
+  />
 </robot>
